File: Kimiro.kicad_sch (KiCad schematic)
At the start: 27 parts, among them J2 USB_C_Left, J3 Left, J4 Right, Q1 AO3407, U1 ProMicro, U2 TP4054, U3 MS88FS3, U4 XC6220B331MR

Commit message: Kicad PCB design ver 1.1
Parts:
- removed D1: 1N5819, Diode_SMD:D_SOD-323F, symbol nrfmicro-rescue:MBR0520
- removed D3: RED, LED_SMD:LED_0603_1608Metric, symbol Device:LED
- removed Q1: AO3407, Package_TO_SOT_SMD:SOT-23, symbol nrfmicro-rescue:BSS83P
- removed R3: 100K, Resistor_SMD:R_0402_1005Metric, symbol nrfmicro-rescue:R
- removed R4: 1K, Resistor_SMD:R_0402_1005Metric, symbol nrfmicro-rescue:R
- removed R5: RPROG, Resistor_SMD:R_0402_1005Metric, symbol nrfmicro-rescue:R
- removed U1: ProMicro, symbol keebio:ProMicro
- removed U2: TP4054, Package_TO_SOT_SMD:SOT-23-5, symbol Battery_Management:MCP73832-2-OT
- added C2, C3: 4.7uF, Capacitor_SMD:C_0402_1005Metric, symbol Device:C_Small
- added D1: RED, LED_SMD:LED_0603_1608Metric, symbol Device:LED_Small
- added R3, R4, R6: 10k, Resistor_SMD:R_0402_1005Metric, symbol Device:R_Small
- added R5: 3.9k, Resistor_SMD:R_0402_1005Metric, symbol Device:R_Small
- added TP1, TP10, TP2, TP3, TP4, TP5, TP6, TP7, TP8, TP9: TestPoint, TestPoint:TestPoint_Pad_1.5x1.5mm, symbol Connector:TestPoint
- added U1: BQ24075RGT, Package_DFN_QFN:VQFN-16-1EP_3x3mm_P0.5mm_EP1.6x1.6mm, symbol Battery_Management:BQ24075RGT
- C1: value 10uF -> 1uF; Digikey (none) -> 1276-1067-1-ND; JLC Part C19702 -> C52923; LCSC Part C19702 -> C52923; Manufacturer Part CL10A106KP8NNNC -> CL05A105KO5NNNC
- J1: renamed from J2; footprint kien242:USB-C-Low -> footprints:USB-C_C168688
- J2: renamed from J3; footprint Sakura-library:Conn_1x13_P2.54mm -> Kimiro-library:Conn_1x13_P2.54mm
- J3: renamed from J4; footprint Sakura-library:Conn_1x13_P2.54mm -> Kimiro-library:Conn_1x13_P2.54mm
- renumbered C5 to C4, C6 to C5, C8 to C6, R11 to R10, R8 to R7, R9 to R8, R10 to R9, U3 to U2, U4 to U3
Connections:
- net BATTERY_PIN: now also U2.11 (0.28/AIN4)
- net CHARGE_CTRL_1: now also R4.1
- net CHARGE_CTRL_2: now also R5.2
- net GND: now also C1.2, U2.34 (GND), C2.2, C3.1, R3.2, U1.15 (SYSOFF), U1.17 (VSS), U1.4 (~{CE}), U1.5 (EN2), U1.8 (VSS); no longer C1.1
- net VBAT: now also J3.2 (Pin_2), C3.2, U1.2 (BAT), U1.3 (BAT)
- net VBUS: now also C1.1, U1.13 (IN); no longer C1.2
- net VDDH: now also C2.1, R6.1, U1.10 (OUT), U1.11 (OUT), U1.6 (EN1)
- net P0.20: now reaches J2.10 (Pin_10)
- net P0.20: now also U2.44 (*0.20)
- net P0.22: now reaches J2.11 (Pin_11)
- net P0.22: now also U2.45 (*0.22)
- net P0.24: now reaches J2.12 (Pin_12)
- net P0.24: now also U2.46 (*0.24)
- net P1.00: now reaches J2.13 (Pin_13)
- net P1.00: now also U2.47 (*1.00)
- net P0.19: now reaches J2.2 (Pin_2)
- net P0.19: now also U2.38 (*0.19)
- net P0.13: now reaches J2.3 (Pin_3)
- net P0.13: now also U2.39 (*0.13)
- net P0.15: now reaches J2.6 (Pin_6)
- net P0.15: now also U2.40 (*0.15)
- net P0.17: now reaches J2.7 (Pin_7)
- net P0.17: now also U2.41 (*0.17)
- net P0.21: now reaches J2.8 (Pin_8)
- net P0.21: now also U2.42 (*0.21)
- net P0.23: now reaches J2.9 (Pin_9)
- net P0.23: now also U2.43 (*0.23)
- net P0.29: now reaches U2.10 (0.29/AIN5)
- net P0.30: now reaches U2.12 (0.30/AIN6)
- net P0.30: now also TP6.1
- net P0.31: now reaches U2.13 (0.31/AIN7)
- net P0.31: now also TP9.1
- net P0.27: now reaches U2.14 (0.27*)
- net P0.27: now also J3.10 (Pin_10)
- net P0.05: now reaches U2.15 (0.05*/AIN3)
- net P0.05: now also J3.6 (Pin_6)
- net P0.04: now reaches U2.16 (0.04*/AIN2)
- net P0.04: now also J3.7 (Pin_7)
- net P0.26: now reaches U2.17 (0.26*)
- net P0.26: now also J3.11 (Pin_11)
- net P0.07: now reaches U2.19 (0.07*)
- net P0.07: now also J3.12 (Pin_12)
- net P1.11: now reaches U2.2 (1.11)
- net P0.06: now reaches U2.20 (0.06*)
- net P0.06: now also J3.13 (Pin_13)
- net P1.08: now reaches U2.21 (1.08*)
- net P1.08: now also TP5.1
- net P0.11: now reaches U2.22 (0.11*)
- net P0.11: now also TP2.1
- net P0.08: now reaches U2.25 (0.08*)
- net P0.08: now also TP3.1
- net P1.09: now reaches U2.26 (1.09*)
- net P1.09: now also TP1.1
- net P0.12: now reaches U2.27 (0.12*)
- net P0.12: now also TP4.1
- net P1.12: now reaches U2.3 (1.12)
- net P1.10: now reaches U2.4 (1.10)
- net P0.25: now reaches U2.48 (*0.25)
- net P1.14: now reaches U2.5 (1.14)
- net P1.14: now also TP7.1
- net P0.03: now reaches U2.6 (0.03/AIN1)
- net P0.03: now also J3.8 (Pin_8)
- net P1.13: now reaches U2.7 (1.13)
- net P1.13: now also TP8.1
- net P1.15: now reaches U2.8 (1.15)
- net P1.15: now also TP10.1
- net P0.02: now reaches U2.9 (0.02/AIN0)
- net P0.02: now also J3.9 (Pin_9)
- net LED renamed BLUE_LED
- new net: D1.2 (A), R6.2
- new net: R3.1, U1.1 (TS)
- new net: R4.2, R5.1, U1.16 (ISET)
- new net: D1.1 (K), U1.9 (~{CHG})
- no-connect marks 4 -> 17
Other:
- note added: "Z, Z: 0mA (off) 0, Z: 100mA Z, 0: 250mA 0, 0: 350mA"
- note removed: "RProg = 1000/iBat iBat in amps RProg iBAT 10k 100mA 5k 200mA 2.5k 400mA 2k 500mA 1.25k 800mA"
- moved on the sheet: C4, C5, R9, U3
